Commit message: lab2

File: lab2/urdf/movable.urdf (robot description, URDF)
Before this commit: robot manipulator, 5 links, 4 joints
Links:
- link hand: geometry visual mesh filename=package://lab2/hand.obj scale=0.05 0.05 0.1
- link link_1: geometry visual cylinder length=${params['s1']['l_len']} radius=${l_width}
- link link_2: geometry visual cylinder length=${params['s2']['l_len']} radius=${l_width}
- link link_3: geometry visual cylinder length=${params['s3']['l_len']} radius=${l_width}
Joints:
- joint base_to_link1: origin xyz=${props['i1']['j_xyz']} rpy=${props['i1']['j_rpy']} -> xyz=${params['s1']['j_xyz']} rpy=${params['s1']['j_rpy']}; type fixed -> prismatic
- joint link1_to_link2: origin xyz=${props['i2']['j_xyz']} rpy=${props['i2']['j_rpy']} -> xyz=${params['s2']['j_xyz']} rpy=${params['s2']['j_rpy']}; type fixed -> prismatic
- joint link2_to_link3: origin xyz=${props['i3']['j_xyz']} rpy=${props['i3']['j_rpy']} -> xyz=${params['s3']['j_xyz']} rpy=${params['s3']['j_rpy']}; type fixed -> prismatic

File: lab2/urdf/nonmovable.urdf (robot description, URDF)
Before this commit: robot manipulator, 5 links, 4 joints
Links:
- link hand: geometry visual mesh filename=package://lab2/hand.obj scale=0.05 0.05 0.1
- link link_1: geometry visual cylinder length=${params['s1']['l_len']} radius=${l_width}
- link link_2: geometry visual cylinder length=${params['s2']['l_len']} radius=${l_width}
- link link_3: geometry visual cylinder length=${params['s3']['l_len']} radius=${l_width}
Joints:
- joint base_to_link1: origin xyz=${props['i1']['j_xyz']} rpy=${props['i1']['j_rpy']} -> xyz=${params['s1']['j_xyz']} rpy=${params['s1']['j_rpy']}
- joint link1_to_link2: origin xyz=${props['i2']['j_xyz']} rpy=${props['i2']['j_rpy']} -> xyz=${params['s2']['j_xyz']} rpy=${params['s2']['j_rpy']}
- joint link2_to_link3: origin xyz=${props['i3']['j_xyz']} rpy=${props['i3']['j_rpy']} -> xyz=${params['s3']['j_xyz']} rpy=${params['s3']['j_rpy']}
